File: CAN_module/can_module_top.kicad_sch (KiCad schematic)
At the start: 33 parts, among them IC1 SN65HVD233QDRQ1, J2 Barrel_Jack_Switch, J3 Screw_Terminal_01x02, J4 Conn_Coaxial, U1 PC817, U2 LM5164QDDATQ1, U3 Antena BT - 2450AT42E010B001E

Commit message: Add files via upload
Parts:
- removed J3: Screw_Terminal_01x02, Antyradar_footprints:CUI_TB002-500-02BE, symbol Antiradar:Screw_Terminal_01x02
- removed R6: 10 Ohm, Resistor_SMD:R_0805_2012Metric, symbol Antiradar:RES_10_OHM_10%_1/4W_0805
- removed U2: LM5164QDDATQ1, Package_SO:HSOP-8-1EP_3.9x4.9mm_P1.27mm_EP2.41x3.1mm_ThermalVias, symbol Antiradar:LM5164DDA
- added C12: 100nF, Capacitor_SMD:C_0805_2012Metric, symbol Antiradar:C_100nF_10%_16V
- added C13: 47uF, Antyradar_footprints:CAPC6153X670N, symbol Antiradar:C_47uF_20%_50V_6050_X7R
- added C14: 1nF, Capacitor_SMD:C_0201_0603Metric, symbol Antiradar:C_1nF_10%_50V_X7R_0603
- added C15: 240pF, Capacitor_SMD:C_01005_0402Metric, symbol Antiradar:C_240pF_1%_50V_0402
- added C2, C3: 2.2uF, SCK_Footprints:C_0805_2012Metric_Pad1.18x1.45mm_HandSolder, symbol Antiradar:C_2.2uF_10%_50V_0805_X7R
- added J5: Screw_Terminal_01x02, Antyradar_footprints:CUI_TB002-500-02BE, symbol Antiradar:Screw_Terminal_01x02
- added L1: 47uH, Antyradar_footprints:NRS8040T470MJGK, symbol Antiradar:L_47uH_20%_100KHz_1.5A_0.182Ohm_8040
- added R1: 330Ω, Resistor_SMD:R_0805_2012Metric, symbol Antiradar:RES_330_10%_1/4W_0805
- added R10, R8: 56kΩ, Resistor_SMD:R_0805_2012Metric, symbol Antiradar:RES_56k_1%_1/2W_0805
- added R11: 30kΩ, Resistor_SMD:R_0805_2012Metric, symbol Antiradar:RES_30k_1%_1/4W_0805
- added R2: 10kΩ, Resistor_SMD:R_0805_2012Metric, symbol Antiradar:RES_10k_10%_1/4W_0805
- added R6: 10Ω, Resistor_SMD:R_0805_2012Metric, symbol Antiradar:RES_10_10%_1/4W_0805
- added R7: 27.4kΩ, Resistor_SMD:R_0805_2012Metric, symbol Antiradar:RES_27.4k_0.5%_1/4W_0805
- added R9: 100kΩ, Resistor_SMD:R_0805_2012Metric, symbol Antiradar:RES_100k_1%_1/2W_0805
- added U2: LM5164QDDATQ1, Package_SO:HSOP-8-1EP_3.9x4.9mm_P1.27mm_EP2.41x3.1mm_ThermalVias, symbol Antiradar:LM5164DDATAQ1
- R3, R4: value 10k -> 10kΩ
- R5: value 1k -> 1kΩ
Connections:
- net +3.3V: now also C13.1, C14.2, L1.2, R10.2, R2.1, R9.1
- net GND: now also U1.3, C12.1, C13.2, C2.2, R7.2, R8.2, U2.9 (PAD)
- net VCC_REF: now also R6.2
- net at JP1.1 (A): now also R4.1; no longer R4.2
- net at GREEN1.2 (A): now also R4.2; no longer R4.1
- net at J2.1: now also C12.2, C2.1, U2.2 (VIN), U2.3 (EN/UVLO)
- net at J2.2: now also U2.1 (GND)
- net at C11.2, C9.2, L3.2: now also R6.1
- net AR_IN: now reaches MCU1.8 (PTA0)
- net AR_IN: now also U1.4, R2.2
- net at U1.1: now also R1.2
- net at U1.2: now also J5.2 (Pin_2)
- new net: C15.1, R8.1, R9.2, U2.5 (FB)
- new net: C3.1, L1.1, R11.1, U2.8 (SW)
- new net: C3.2, U2.7 (BST)
- new net: R7.1, U2.4 (RON)
- new net: J5.1 (Pin_1), R1.1
- new net: C14.1, C15.2, R11.2
- new net: R10.1, U2.6 (PGOOD)
- no-connect marks 11 -> 12
Other:
- moved on the sheet: C4, C7, C8, J2, MCU1, U1, XTAL1

Commit message: Add files via upload
Parts:
- added C16, C17, C18, C19, C20, C21, C22, C23, C24: 100nF, Capacitor_SMD:C_0805_2012Metric, symbol Antiradar:C_100nF_10%_16V
- C10: footprint https://mm.digikey.com/Volume0/opasdata/d220001/medias/docus/1105/CL21B105KAFNNNE_Spec.pdf -> SCK_Footprints:C_0805_2012Metric_Pad1.18x1.45mm_HandSolder
- L3: footprint LED_SMD:LED_0402_1005Metric -> Inductor_SMD:L_0402_1005Metric
- renumbered GNSS_module to GNSS_module1
Connections:
- net +3.3V: now also GNSS_module1.7 (VDD_USB), MCU1.21 (VDD_IO_D/VDD_DCDC), MCU1.29 (VDD_ANA), MCU1.4 (VDD_IO_ABC), MCU1.41 (VDD_CORE), MCU1.6 (VDD_SWITCH), C16.1, C19.1, C21.1, C23.1, C24.1
- net GND: now also MCU1.19 (VSS_DCDC), MCU1.49 (VSS), C16.2, C17.2, C18.2, C19.2, C20.2, C21.2, C22.2, C23.2, C24.2; no longer GNSS_module1.7 (VDD_USB)
- net at MCU1.15 (VDD_LDO_CORE): now also C18.1
- net at MCU1.16 (VOUT_CORE/VDD_CORE): now also C17.1
- net at MCU1.22 (VOUT_SYS/VDD_SYS): now also C20.1
- net at MCU1.7 (VOUT_SWITCH): now also C22.1
- no-connect marks 12 -> 35
Other:
- moved on the sheet: J5, R1, R2, U1

Commit message: Add files via upload
Other:
- company: (none) -> Tobiasz Kobza; Mikołaj Krok; Adam Michalik
- title: (none) -> Schemat elektroniczny modułu PCB antyradar-CAN
- moved on the sheet: C16, C17, C18, C19, C20, C21, C22, C23, C24, C4, C7, C8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

Commit message: Add files via upload
Parts:
- removed U3: Antena BT - 2450AT42E010B001E, Antyradar_footprints:2450AT42E010B_JOT, symbol Antiradar:2450AT42E010B001E
- added U3: Ant BT - 2450AT18D0100E, Antyradar_footprints:2450AT18D0100E_JOT, symbol Antiradar:Antenna BT - 2450AT18D0100E
Connections:
- net GND: now also U3.2 (GND), U3.3 (GND), U3.4 (GND/FEED)
- net at C6.2: now also U3.1 (FEED/GND)
Changed lines of the file:
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@@
 	)
 	(junction
-		(at 276.86 30.48)
-		(diameter 0)
-		(color 0 0 0 0)
-	)
-	(junction
 		(at 243.84 127)
 		(diameter 0)
@@
 	)
 	(junction
+		(at 276.86 30.48)
+		(diameter 0)
+		(color 0 0 0 0)
+	)
+	(junction
 		(at 22.86 185.42)
 		(diameter 0)
@@
 	)
 	(symbol
-		(lib_id "Antiradar:2450AT42E010B001E")
-		(at 220.98 27.94 0)
-		(unit 1)
-		(body_style 1)
-		(exclude_from_sim no)
-		(in_bom yes)
-		(on_board yes)
-		(in_pos_files yes)
-		(dnp no)
-		(fields_autoplaced yes)
-		(property "Reference" "U3"
-			(at 248.92 17.78 0)
-			(show_name no)
-			(do_not_autoplace no)
-			(effects
-				(font
-					(size 1.524 1.524)
-				)
-			)
-		)
-		(property "Value" "Antena BT - 2450AT42E010B001E"
-			(at 248.92 20.32 0)
-			(show_name no)
-			(do_not_autoplace no)
-			(effects
-				(font
-					(size 1.524 1.524)
-				)
-			)
-		)
-		(property "Footprint" "Antyradar_footprints:2450AT42E010B_JOT"
-			(at 220.98 27.94 0)
-			(hide yes)
-			(show_name no)
-			(do_not_autoplace no)
-			(effects
-				(font
-					(size 1.27 1.27)
-					(italic yes)
-				)
-			)
-		)
-		(property "Datasheet" "2450AT42E010B001E"
-			(at 220.98 27.94 0)
-			(hide yes)
-			(show_name no)
-			(do_not_autoplace no)
-			(effects
-				(font
-					(size 1.27 1.27)
-					(italic yes)
-				)
-			)
-		)
-		(property "Description" ""
-			(at 220.98 27.94 0)
-			(hide yes)
-			(show_name no)
-			(do_not_autoplace no)
-			(effects
-				(font
-					(size 1.27 1.27)
-				)
-			)
-		)
-		(pin "3"
-		)
-		(pin "4"
-		)
-		(pin "1"
-		)
-		(pin "2"
-		)
-		(instances
-			(project "CAN_module"
-				(path "/b2f48ca0-b9f2-43ed-bfaa-cdba7794cee1"
-					(reference "U3")
-					(unit 1)
-				)
-			)
-		)
-	)
-	(symbol
 		(lib_id "power:GND")
 		(at 171.45 115.57 0)
@@
 	)
 	(symbol
+		(lib_id "Antiradar:Antenna BT - 2450AT18D0100E")
+		(at 220.98 27.94 0)
+		(unit 1)
+		(body_style 1)
+		(exclude_from_sim no)
+		(in_bom yes)
+		(on_board yes)
+		(in_pos_files yes)
+		(dnp no)
+		(fields_autoplaced yes)
+		(property "Reference" "U3"
+			(at 248.92 17.78 0)
+			(show_name no)
+			(do_not_autoplace no)
+			(effects
+				(font
+					(size 1.524 1.524)
+				)
+			)
+		)
+		(property "Value" "Ant BT - 2450AT18D0100E"
+			(at 248.92 20.32 0)
+			(show_name no)
+			(do_not_autoplace no)
+			(effects
+				(font
+					(size 1.524 1.524)
+				)
+			)
+		)
+		(property "Footprint" "Antyradar_footprints:2450AT18D0100E_JOT"
+			(at 220.98 27.94 0)
+			(hide yes)
+			(show_name no)
+			(do_not_autoplace no)
+			(effects
+				(font
+					(size 1.27 1.27)
+					(italic yes)
+				)
+			)
+		)
+		(property "Datasheet" "2450AT18D0100E"
+			(at 220.98 27.94 0)
+			(hide yes)
+			(show_name no)
+			(do_not_autoplace no)
+			(effects
+				(font
+					(size 1.27 1.27)
+					(italic yes)
+				)
+			)
+		)
+		(property "Description" ""
+			(at 220.98 27.94 0)
+			(hide yes)
+			(show_name no)
+			(do_not_autoplace no)
+			(effects
+				(font
+					(size 1.27 1.27)
+				)
+			)
+		)
+		(pin "3"
+		)
+		(pin "1"
+		)
+		(pin "4"
+		)
+		(pin "2"
+		)
+		(instances
+			(project "CAN_module"
+				(path "/b2f48ca0-b9f2-43ed-bfaa-cdba7794cee1"
+					(reference "U3")
+					(unit 1)
+				)
+			)
+		)
+	)
+	(symbol
 		(lib_id "power:GND")
 		(at 120.65 69.85 0)
@@
 					(unit 1)
 				)
+			)
+		)
+	)
+	(symbol
+		(lib_id "power:GND")
+		(at 220.98 30.48 0)
+		(mirror y)
+		(unit 1)
+		(body_style 1)
+		(exclude_from_sim no)
+		(in_bom yes)
+		(on_board yes)
+		(in_pos_files yes)
+		(dnp no)
+		(property "Reference" "#PWR054"
+			(at 220.98 36.83 0)
+			(hide yes)
+			(show_name no)
+			(do_not_autoplace no)
+			(effects
+				(font
+					(size 1.27 1.27)
+				)
+			)
+		)
+		(property "Value" "GND"
+			(at 220.98 34.036 0)
+			(show_name no)
+			(do_not_autoplace no)
+			(effects
+				(font
+					(size 1.27 1.27)
+				)
+			)
+		)
+		(property "Footprint" ""
+			(at 220.98 30.48 0)
+			(hide yes)
+			(show_name no)
+			(do_not_autoplace no)
+			(effects
+				(font
+					(size 1.27 1.27)
+				)
+			)
+		)
+		(property "Datasheet" ""
+			(at 220.98 30.48 0)
+			(hide yes)
+			(show_name no)
+			(do_not_autoplace no)
+			(effects
+				(font
+					(size 1.27 1.27)
+				)
+			)
+		)
+		(property "Description" "Power symbol creates a global label with name \"GND\" , ground"
+			(at 220.98 30.48 0)
+			(hide yes)
+			(show_name no)
+			(do_not_autoplace no)
+			(effects
+				(font
+					(size 1.27 1.27)
+				)
+			)
+		)
+		(pin "1"
+		)
+		(instances
+			(project "CAN_module"
+				(path "/b2f48ca0-b9f2-43ed-bfaa-cdba7794cee1"
+					(reference "#PWR054")
+					(unit 1)
+				)
