File: CAN_module/can_module_top.kicad_sch (KiCad schematic)
At the start: 56 parts, among them IC1 SN65HVD233QDRQ1, J2 Barrel_Jack_Switch, J4 Conn_Coaxial, J5 Screw_Terminal_01x02, U1 PC817, U2 LM5164QDDATQ1, U3 Antena BT - 2450AT42E010B001E

Commit message: Add files via upload
Parts:
- removed C5, C6: C, symbol Device:C
- removed L2: L, symbol Device:L
- removed U3: Antena BT - 2450AT42E010B001E, Antyradar_footprints:2450AT42E010B_JOT, symbol Antiradar:2450AT42E010B001E
- added U3: Ant BT - 2450AT18D0100E, Antyradar_footprints:2450AT18D0100E_JOT, symbol Antiradar:Antenna BT - 2450AT18D0100E
Connections:
- net Antenna_BT: now also U3.1 (FEED/GND)
- net GND: now also U3.2 (GND), U3.3 (GND), U3.4 (GND/FEED)
- net CAN_N: now reaches D2.2 (CATHODE_2), IC1.6 (CANL), OBD-II_CONNECTOR1.2
- net CAN_P: now reaches D2.1 (CATHODE_1), IC1.7 (CANH), OBD-II_CONNECTOR1.7
