File: CAN_module/CAN_module.kicad_sch (KiCad schematic)
At the start: 0 parts

Commit message: Add files via upload
Other:
- note added: "CAN0_RX"
- note added: "CAN0_TX"
- note added: "EXTAL"
- note added: "GPIO"
- note added: "RF_IN"
- note added: "VCC 3.3V"
- note added: "VPA_2P4GHZ"
- note added: "XTAL"
- note removed: "UART"
- company: (none) -> Tobiasz Kobza; Mikołaj Krok; Adam Michalik
- title: (none) -> Schemat blokowy modułu PCB antyradar-CAN
